File: displinux/displinux.kicad_sch (KiCad schematic)
At the start: 144 parts, among them J1 USB4105-GF-A, J10 Conn_01x03, J2 USB4105-GF-A, J3 AudioJack4, J4 Conn_02x10_Counter_Clockwise, J5 HR911105A, J6 Conn_01x24_MountingPin, J7 Conn_01x06, J8 Conn_01x40_MountingPin, J9 Conn_01x02_Pin, U1 DP83848C, U2 SY8089AAAC, U3 F133, U4 SY8089AAAC, U5 XC6206P_2_8_MR, U6 XC6206P_1_2_MR, U7 SY7201ABC, U8 W25N01KV, X1 ASE-50MHz, Y1 24M, Y2 Crystal

Commit message: add lvds
Parts:
- removed D3: D, Diode_SMD:D_SOD-523, symbol Device:D
- removed R1, R3: 5.1k, Resistor_SMD:R_0603_1608Metric, symbol Device:R
- removed R51, R52, R53, R54: 10k, Resistor_SMD:R_0603_1608Metric, symbol Device:R
- added C14, C64, C65, C66: 10u, Capacitor_SMD:C_0603_1608Metric, symbol Device:C
- added J11: Conn_01x40_MountingPin, Connector_FFC-FPC:TE_4-1734839-0_1x40-1MP_P0.5mm_Horizontal, symbol Connector_Generic_MountingPin:Conn_01x40_MountingPin
- added R37, R47: 10k, Resistor_SMD:R_0603_1608Metric, symbol Device:R
- added R48: 150K, Resistor_SMD:R_0603_1608Metric, symbol Device:R
- added U9: PAM8301, Package_TO_SOT_SMD:SOT-23-6, symbol Amplifier_Audio:PAM8301
- C37: value 0.1u -> 4.7u
- R2, R4, R5, R6: value 5.1k -> 51k
- R49: value 10k -> 150K
- R50: value 10k -> 2k
Connections:
- net +3V3: now also R50.2, U3.29 (LDO-IN), C14.1, J11.2 (Pin_2), J11.3 (Pin_3), J11.36 (Pin_36), J11.4 (Pin_4), R37.1
- net +5V: now also C64.1, U9.5 (VDD)
- net GND: now also C14.2, C64.2, J11.10 (Pin_10), J11.13 (Pin_13), J11.16 (Pin_16), J11.19 (Pin_19), J11.22 (Pin_22), J11.25 (Pin_25), J11.28 (Pin_28), J11.31 (Pin_31), J11.32 (Pin_32), J11.33 (Pin_33), J11.MP (MountPin), R47.2, U9.2 (GND); no longer R49.2, R50.2
- net HPOUTL: now also C66.1; no longer C6.2
- net HPOUTR: now also C65.1; no longer C4.2
- net LCD0-D10: now also J11.18 (Pin_18)
- net LCD0-D11: now also J11.17 (Pin_17)
- net LCD0-D14: now also J11.21 (Pin_21)
- net LCD0-D15: now also J11.20 (Pin_20)
- net LCD0-D16: no longer R49.1
- net LCD0-D17: no longer R50.1
- net LCD0-D18: now also J11.24 (Pin_24)
- net LCD0-D19: now also J11.23 (Pin_23)
- net LCD0-D2: now also J11.9 (Pin_9)
- net LCD0-D20: now also J11.27 (Pin_27)
- net LCD0-D21: now also J11.26 (Pin_26)
- net LCD0-D22: now also J11.30 (Pin_30)
- net LCD0-D23: now also J11.29 (Pin_29)
- net LCD0-D3: now also J11.8 (Pin_8)
- net LCD0-D4: now also J11.12 (Pin_12)
- net LCD0-D5: now also J11.11 (Pin_11)
- net LCD0-D6: now also J11.15 (Pin_15)
- net LCD0-D7: now also J11.14 (Pin_14)
- net LCD0-HSYNC: now also J11.6 (Pin_6)
- net LCD0-VSYNC: now also J11.7 (Pin_7)
- net LCD_A: now also J11.38 (Pin_38), J11.39 (Pin_39), J11.40 (Pin_40)
- net MIC3N: now also C4.1; no longer J10.3 (Pin_3)
- net MIC3P: now also C6.1; no longer J10.2 (Pin_2)
- net PWM_LCD: now reaches U3.52 (PD22)
- net PWM_LCD: now also J11.35 (Pin_35)
- net at J3.R1: now also U9.1 (OUT-); no longer C4.1
- net at J3.T: now also U9.6 (OUT+); no longer C6.1
- new net: C6.2, J10.2 (Pin_2)
- new net: C66.2, R49.1
- new net: R49.2, U9.4 (~{SD})
- new net: C4.2, J10.3 (Pin_3), R50.1
- new net: C65.2, R48.1
- new net: R48.2, U9.3 (IN)
- new net: J11.5 (Pin_5), R37.2, R47.1
- no-connect marks 34 -> 36
Other:
- note added: "D0_LVDS0-V0P"
- note added: "D10_LVDS1-V0P"
- note added: "D11_LVDS1-V0N"
- note added: "D12_LVDS1-V1P"
- note added: "D13_LVDS1-V1N"
- note added: "D14_LVDS1-V2P"
- note added: "D15_LVDS1-V2N"
- note added: "D16_LVDS1-ClkN"
- note added: "D17_LVDS1-ClkN"
- note added: "D1_LVDS0-V0N"
- note added: "D2_LVDS0-V1P"
- note added: "D3_LVDS0-V1N"
- note added: "D4_LVDS0-V2P"
- note added: "D5_LVDS0-V2N"
- note added: "D6_LVDS0-ClkP"
- note added: "D7_LVDS0-ClkN"
- note added: "EDID clk"
- note added: "EDID data"
- note added: "EDID writing protection"
- note added: "LCD-LVDS"
- note added: "LVDS0-ODD"
- note added: "LVDS1-EVEN"
- note removed: "LCD-MIPI"
- moved on the sheet: C1, C3, C5, C7, J10, J3, J4, J9, R12, R2, R9

Commit message: some fixes
Parts:
- added R1: 10, Resistor_SMD:R_0603_1608Metric, symbol Device:R
- added R3, R51: 51k, Resistor_SMD:R_0603_1608Metric, symbol Device:R
- C64: value 10u -> 470u
- XS1: footprint Connector_Card:microSD_HC_Hirose_DM3AT-SF-PEJM5 -> Micro_SD:J_SD_Card-micro_socket_A
Connections:
- net +5V: now also R1.2; no longer C64.1, U9.5 (VDD)
- net GND: now also R3.1, R51.1
- net at R49.2: now also R48.2, U9.3 (IN); no longer U9.4 (~{SD})
- net at J1.A5 (CC1), R2.2: now also R3.2
- net at J1.B5 (CC2), R4.2: now also R51.2
- new net: C64.1, R1.1, U9.4 (~{SD}), U9.5 (VDD)
Other:
- moved on the sheet: C65, C66, R48, R49

Commit message: fix audio
Parts:
- added R52, R53: 5R1, Resistor_SMD:R_0603_1608Metric, symbol Device:R
- added R54: 0, Resistor_SMD:R_0603_1608Metric, symbol Device:R
- R29: footprint Resistor_SMD:R_0603_1608Metric -> Resistor_SMD:R_0805_2012Metric_Pad1.20x1.40mm_HandSolder
Connections:
- net +3V3: now also R52.1; no longer J8.31 (Pin_31)
- net GND: now also R53.2
- net PWM_LCD: now also R54.1
- net at R33.1, U7.4 (EN/PWM): now also R54.2
- new net DISP: J8.31 (Pin_31), R52.2, R53.1
