File: displinux/displinux.kicad_sch (KiCad schematic)
At the start: 152 parts, among them J1 USB4105-GF-A, J10 Conn_01x03, J11 Conn_01x40_MountingPin, J2 USB4105-GF-A, J3 AudioJack4, J4 Conn_02x10_Counter_Clockwise, J5 HR911105A, J6 Conn_01x24_MountingPin, J7 Conn_01x06, J8 Conn_01x40_MountingPin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

Commit message: change otg CCM1 CCM2 res
Parts:
- R3, R4: value 51k -> 5.1k
Changed lines of the file:
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@@
 			)
 		)
-		(property "Value" "51k"
+		(property "Value" "5.1k"
 			(at 463.55 20.32 90)
 			(effects
@@
 			)
 		)
-		(property "Value" "51k"
+		(property "Value" "5.1k"
 			(at 506.73 20.32 90)
 			(effects
